File: Carrier Board.sch (EAGLE design)
At the start: 62 parts, among them J1 S2B-PH-SM4-TB(LF)(SN), J2 S2B-PH-SM4-TB(LF)(SN), J3 BM04B-SRSS-TB(LF)(SN), J4 BM06B-SRSS-TB(LF)(SN), J5 BM06B-SRSS-TB(LF)(SN), J6 BM06B-SRSS-TB(LF)(SN), J7 BM04B-SRSS-TB(LF)(SN), J8 BM04B-SRSS-TB(LF)(SN), J9 BM04B-SRSS-TB(LF)(SN), P1 Particle Boron / Xenon / Argon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

Commit message: Updated for Macrofab
Parts:
- removed H1, H2, H3, H4: STAND-OFF-M2.5, Custom Components:STAND-OFF-M2.5
- removed Q1: 2N7002L, Carrier Board:2N7002L
- removed U2: MB85RC64, Fujitsu_By_element14_Batch_1:MB85RC128PNF-G-JNE1
- added Q2: BSS138, Custom Components:BSS138
- added U7: MB85RC64TA, Custom Components:MB85RC64TA
- C1, C6, C7, C9: device SparkFun-Capacitors:CAP0805 -> Custom Components:CAP-MF-0.1UF-0805
- C10, C4, C5: device SparkFun-Capacitors:CAP0805 -> Custom Components:CAP-10NF-0805
- C11: device SparkFun-Capacitors:CAP0805 -> Custom Components:CAP-47PF-0805
- C2, C3: device SparkFun-Capacitors:CAP0805 -> Custom Components:CAP-MF-1UF-0805
- F1: value 63V/1.5A -> 6V/0.5A
- J3, J7, J8, J9: value BM04B-SRSS-TB(LF)(SN) -> BM04B-SRSS-TBT(LF)(SN)
- J4, J5, J6: value BM06B-SRSS-TB(LF)(SN) -> BM06B-SRSS-TBT(LF)(SN); device Custom Components:BM06B-SRSS-TB(LF)(SN) -> Custom Components:BM06B-SRSS-TBT(LF)(SN)
- P1: device Carrier Board:PARTICLE-DEVICES-BORON -> Custom Components:PARTICLE-DEVICES-BORON
- R1, R6: device SparkFun-Passives:RESISTOR0805-RES -> Custom Components:RESISTOR-MF-100K-0805
- R4, R5: device SparkFun-Passives:RESISTOR0805-RES -> Custom Components:RESISTOR-MF-4.7K-0805
- R7: device SparkFun-Passives:RESISTOR0805-RES -> Custom Components:RESISTOR-MF-10K-0805
- R8, R9: device SparkFun-Passives:RESISTOR0805-RES -> Custom Components:RESISTOR-MF-100-0805
- U1: device TMP36:TMP36GRTZ-REEL7 -> Custom Components:TMP36GRTZ-REEL7
- U3: device Carrier Board:AB1805-T3 -> Custom Components:AB1805-T3
- U6: device Carrier Board:XC6215B332MR-G -> Custom Components:XC6215B332MR-G
- Y1: device Carrier Board:ABS07-120-32.768KHZ-T -> Custom Components:ABS07-120-32.768KHZ-T
Connections:
- net EN: now also Q2.DRAIN; no longer Q1.DRAIN
- net GND: now also Q2.SOURCE, U7.A0, U7.A1, U7.A2, U7.VSS, U7.WP; no longer Q1.SOURCE, U2.A0, U2.A1, U2.A2, U2.VSS, U2.WP
- net PSW: now also Q2.GATE; no longer Q1.GATE
- net SCL: now also U7.SCL; no longer U2.SCL
- net SDA: now also U7.SDA; no longer U2.SDA
- net VCC: now also U7.VDD; no longer U2.VDD
Other:
- note added: "Based on this Application Note https://github.com/particle-iot/app-notes/tree/master/AN023-Watchdog-Timers"
- note removed: "Add connector for external Reset and LED"
- note removed: "Particle Boron / Argon / Xenon Carrier Board"

Commit message: Latest Version
Parts:
- C11: value 47pF -> GRM21A5C2D470JW01D; device Custom Components:CAP-47PF-0805 -> Custom Components:GRM21A5C2D470JW01D; HOUSEPART YES -> (none); MPN MF-CAP-0805-0.1uF -> (none); POPULATE 1 -> (none)
- J1, J2: value S2B-PH-SM4-TB(LF)(SN) -> B2B-PH-SM4-TB(LF)(SN); device SparkFun-Connectors:JST_2MM_MALE -> Custom Components:B2B-PH-SM4-TB(LF)(SN); MFG JST S2B-PH-SM4-TB(LF)(SN) -> (none)
Connections:
- net BATT-IN: now also J1.1; no longer J2.+
- net DC-IN: now also D3.C, J2.1; no longer J1.+, JP7.1
- net GND: now also C11.1, J1.2, J2.2, JP7.1; no longer C11.2, D3.A, J1.-, J2.-
- net N$1: now also D3.A; no longer D3.C
- net N$11: now also C11.2; no longer C11.1
Other:
- moved on the sheet: C11, D3

Commit message: Updated FRAM footprint to address stock issue
Parts:
- U7: value MB85RC64TA -> MB85RC64TASON8; device Custom Components:MB85RC64TA -> Custom Components:MB85RC64TASON8
Other:
- note added: "v1.6a"
- note removed: "v1.4"
- moved on the sheet: U7
Changed lines of the file:
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@@
 <grid distance="0.1" unitdist="inch" unit="inch" style="lines" multiple="1" display="no" altdistance="0.01" altunitdist="inch" altunit="inch"/>
 <layers>
-<layer number="1" name="Top" color="4" fill="1" visible="no" active="no"/>
-<layer number="2" name="Route2" color="1" fill="3" visible="no" active="no"/>
-<layer number="15" name="Route15" color="4" fill="6" visible="no" active="no"/>
-<layer number="16" name="Bottom" color="1" fill="1" visible="no" active="no"/>
-<layer number="17" name="Pads" color="2" fill="1" visible="no" active="no"/>
-<layer number="18" name="Vias" color="2" fill="1" visible="no" active="no"/>
-<layer number="19" name="Unrouted" color="6" fill="1" visible="no" active="no"/>
-<layer number="20" name="Dimension" color="15" fill="1" visible="no" active="no"/>
-<layer number="21" name="tPlace" color="7" fill="1" visible="no" active="no"/>
-<layer number="22" name="bPlace" color="7" fill="1" visible="no" active="no"/>
-<layer number="23" name="tOrigins" color="15" fill="1" visible="no" active="no"/>
-<layer number="24" name="bOrigins" color="15" fill="1" visible="no" active="no"/>
-<layer number="25" name="tNames" color="7" fill="1" visible="no" active="no"/>
-<layer number="26" name="bNames" color="7" fill="1" visible="no" active="no"/>
-<layer number="27" name="tValues" color="7" fill="1" visible="no" active="no"/>
-<layer number="28" name="bValues" color="7" fill="1" visible="no" active="no"/>
+<layer number="1" name="Top" color="4" fill="1" visible="yes" active="no"/>
+<layer number="2" name="Route2" color="1" fill="3" visible="yes" active="no"/>
+<layer number="15" name="Route15" color="4" fill="6" visible="yes" active="no"/>
+<layer number="16" name="Bottom" color="1" fill="1" visible="yes" active="no"/>
+<layer number="17" name="Pads" color="2" fill="1" visible="yes" active="no"/>
+<layer number="18" name="Vias" color="2" fill="1" visible="yes" active="no"/>
+<layer number="19" name="Unrouted" color="6" fill="1" visible="yes" active="no"/>
+<layer number="20" name="Dimension" color="15" fill="1" visible="yes" active="no"/>
+<layer number="21" name="tPlace" color="7" fill="1" visible="yes" active="no"/>
+<layer number="22" name="bPlace" color="7" fill="1" visible="yes" active="no"/>
+<layer number="23" name="tOrigins" color="15" fill="1" visible="yes" active="no"/>
+<layer number="24" name="bOrigins" color="15" fill="1" visible="yes" active="no"/>
+<layer number="25" name="tNames" color="7" fill="1" visible="yes" active="no"/>
+<layer number="26" name="bNames" color="7" fill="1" visible="yes" active="no"/>
+<layer number="27" name="tValues" color="7" fill="1" visible="yes" active="no"/>
+<layer number="28" name="bValues" color="7" fill="1" visible="yes" active="no"/>
 <layer number="29" name="tStop" color="7" fill="3" visible="no" active="no"/>
 <layer number="30" name="bStop" color="7" fill="6" visible="no" active="no"/>
@@
 <layer number="35" name="tGlue" color="7" fill="4" visible="no" active="no"/>
 <layer number="36" name="bGlue" color="7" fill="5" visible="no" active="no"/>
-<layer number="37" name="tTest" color="7" fill="1" visible="no" active="no"/>
-<layer number="38" name="bTest" color="7" fill="1" visible="no" active="no"/>
+<layer number="37" name="tTest" color="7" fill="1" visible="yes" active="no"/>
+<layer number="38" name="bTest" color="7" fill="1" visible="yes" active="no"/>
 <layer number="39" name="tKeepout" color="4" fill="11" visible="no" active="no"/>
 <layer number="40" name="bKeepout" color="1" fill="11" visible="no" active="no"/>
@@
 <layer number="44" name="Drills" color="7" fill="1" visible="no" active="no"/>
 <layer number="45" name="Holes" color="7" fill="1" visible="no" active="no"/>
-<layer number="46" name="Milling" color="3" fill="1" visible="no" active="no"/>
-<layer number="47" name="Measures" color="7" fill="1" visible="no" active="no"/>
-<layer number="48" name="Document" color="7" fill="1" visible="no" active="no"/>
-<layer number="49" name="Reference" color="7" fill="1" visible="no" active="no"/>
-<layer number="50" name="dxf" color="7" fill="1" visible="no" active="no"/>
-<layer number="51" name="tDocu" color="7" fill="1" visible="no" active="no"/>
-<layer number="52" name="bDocu" color="7" fill="1" visible="no" active="no"/>
-<layer number="53" name="tGND_GNDA" color="7" fill="9" visible="no" active="no"/>
-<layer number="54" name="bGND_GNDA" color="1" fill="9" visible="no" active="no"/>
-<layer number="56" name="wert" color="7" fill="1" visible="no" active="no"/>
-<layer number="57" name="tCAD" color="7" fill="1" visible="no" active="no"/>
-<layer number="59" name="tCarbon" color="7" fill="1" visible="no" active="no"/>
-<layer number="60" name="bCarbon" color="7" fill="1" visible="no" active="no"/>
+<layer number="46" name="Milling" color="3" fill="1" visible="yes" active="no"/>
+<layer number="47" name="Measures" color="7" fill="1" visible="yes" active="no"/>
+<layer number="48" name="Document" color="7" fill="1" visible="yes" active="no"/>
+<layer number="49" name="Reference" color="7" fill="1" visible="yes" active="no"/>
+<layer number="50" name="dxf" color="7" fill="1" visible="yes" active="no"/>
+<layer number="51" name="tDocu" color="7" fill="1" visible="yes" active="no"/>
+<layer number="52" name="bDocu" color="7" fill="1" visible="yes" active="no"/>
+<layer number="53" name="tGND_GNDA" color="7" fill="9" visible="yes" active="no"/>
+<layer number="54" name="bGND_GNDA" color="1" fill="9" visible="yes" active="no"/>
+<layer number="56" name="wert" color="7" fill="1" visible="yes" active="no"/>
+<layer number="57" name="tCAD" color="7" fill="1" visible="yes" active="no"/>
+<layer number="59" name="tCarbon" color="7" fill="1" visible="yes" active="no"/>
+<layer number="60" name="bCarbon" color="7" fill="1" visible="yes" active="no"/>
 <layer number="88" name="SimResults" color="9" fill="1" visible="no" active="no"/>
 <layer number="89" name="SimProbes" color="9" fill="1" visible="no" active="no"/>
@@
 </part>
 <part name="Q2" library="Custom Components" deviceset="BSS138" device=""/>
-<part name="U7" library="Custom Components" deviceset="MB85RC64TA" device=""/>
+<part name="U7" library="Custom Components" deviceset="MB85RC64TA" device="SON8" value="MB85RC64TASON8"/>
 <part name="J1" library="Custom Components" deviceset="B2B-PH-SM4-TB(LF)(SN)" device=""/>
 <part name="J2" library="Custom Components" deviceset="B2B-PH-SM4-TB(LF)(SN)" device=""/>
@@
 <text x="172.72" y="7.62" size="1.778" layer="94">Chip McClelland
 chip@mcclellands.org</text>
-<text x="236.22" y="7.62" size="2.54" layer="94">v1.4</text>
+<text x="236.22" y="7.62" size="2.54" layer="94">v1.6a</text>
 <text x="147.32" y="38.1" size="1.778" layer="94">Power either with DC source or Solar Panel - JST connector
 1) External Power: 5V DC @ 2A
@@
 <text x="86.36" y="177.8" size="2.54" layer="94" ratio="10">Particle Boron / Argon / Xenon Carrier Board - Power Control</text>
 <text x="175.26" y="10.16" size="2.54" layer="94">Chip McClelland</text>
-<text x="236.22" y="7.62" size="2.54" layer="94">v1.4</text>
+<text x="236.22" y="7.62" size="2.54" layer="94">v1.6a</text>
 <text x="93.98" y="116.84" size="1.778" layer="94">Device TPS62291 has
 short circuit protection.
@@
 <text x="172.72" y="7.62" size="1.778" layer="94">Chip McClelland
 chip@mcclellands.org</text>
-<text x="236.22" y="7.62" size="2.54" layer="94">v1.4</text>
+<text x="236.22" y="7.62" size="2.54" layer="94">v1.6a</text>
 <text x="33.02" y="73.66" size="1.778" layer="91">RTC 3.3 Regulator
 200mA Max

Commit message: Fully functional
Parts:
- removed C5: 10nF, Custom Components:CAP-10NF-0805
- removed J3, J8: BM04B-SRSS-TBT(LF)(SN), Custom Components:BM04B-SRSS-TBT(LF)(SN)
- removed U4, U5: TPS22810, Custom Components:TPS22810
- added C12: 0.1uF, Custom Components:CAP-MF-0.1UF-0805
- added FRAME4: FRAME-LETTERNO_PACKAGE, SparkFun-Aesthetics:FRAME-LETTERNO_PACKAGE
- added J10: U.FL-R-SMT(10), Connectors:U.FL-R-SMT(10)
- added Q1, Q3: BSS215P, Custom Components:BSS215P
- added R2, R3: 100k, Custom Components:RESISTOR-MF-100K-0805
- added U2: RFM95CW-915S2, Custom Components:RFM95W-868S2
- C4: value 10nF -> 10uF; device Custom Components:CAP-10NF-0805 -> Custom Components:CAP-MF-10UF-1206; HOUSEPART No -> (none); MPN 08051C103K4T2A -> (none); POPULATE 1 -> (none)
- R8: value 100 -> 100k; device Custom Components:RESISTOR-MF-100-0805 -> Custom Components:RESISTOR-MF-100K-0805; HOUSEPART Yes -> (none); MPN MF-RES-0805-100 -> (none)
Connections:
- removed net D2: G1.5, J4.6, P1.D2
- removed net EN/UVLO: C4.1, C5.1, S1.2, U4.EN/UVLO, U5.EN/UVLO
- removed net MD: P1.MD
- removed net N$10: C7.1, U4.CT
- removed net N$6 (its old number): R8.1, U5.QOD
- removed net N$7: F1.1, R8.2, U5.VOUT
- new net LORA-ANT: J10.1, U2.ANT
- new net ON/OFF: Q1.GATE, Q3.GATE, R2.1, S1.2
- new net RFM-INT: G1.5, J4.6, P1.D2, U2.DIO0
- new net RFM-RST: P1.D6, R8.1, U2.RESET
- new net RFM-SS: P1.D5, R3.1, U2.NSS
- net BATT-IN: now also Q1.SOURCE; no longer U4.VIN
- net DC-IN: now also Q3.SOURCE; no longer U5.VIN
- net GND: now also C12.2, C4.P$2, J10.2, J10.3, R9.1, U2.GND, U2.GND@1, U2.GND@2; no longer C4.2, C5.2, J3.1, J3.SHIELD, J8.1, J8.SHIELD, S1.3, U4.GND, U5.GND
- net LI+: now also C7.1, Q1.DRAIN; no longer R9.2, U4.VOUT
- net MISO: now also U2.MISO
- net MOSI: now also U2.MOSI
- net N$12: now also R9.2, S1.3; no longer R9.1, U4.QOD
- net N$5: now also F1.1, Q3.DRAIN; no longer U5.CT
- net N$9: now also R2.2
- net SCK: now also U2.SCK
- net SCL: no longer J3.4, J8.4
- net SDA: no longer J3.3, J8.3
- net VCC: now also C12.1, C4.P$1, R3.2, R8.2, U2.3_3V
- net VCC2-EXT: no longer J3.2, J8.2
Other:
- note added: "1.5 - Changed to AB1805 for RTC and Watchdog - Major Change 1.6 - Reduced the number of Qwiic connectors - Minor Change 1.6a - Changed to vertical input for JST connectors - Minor Change 1.7 - Changed high-side switching from TI TPS22810 to P-MOSFET BSS215P and the Crystal- Minor Change 1.8 - Added an RFM-95CW LoRA modul to the carrier board. Also, went back to original crystal"
- note added: "CHANGE LOG"
- note added: "Operating Instructions: Note - Power is on when SW1 is connected to Ground. Power is off when SW1 is connected to Batt-IN / LiPO"
- note added: "v1.7"
- note removed: "Device TPS62291 has short circuit protection. Vin is protected by F1"
- note removed: "v1.6a"
